Commit message: update for femto_height

File: wpr2_description/urdf/plan_dual_arms.urdf.xacro (robot description, xacro)
@@ -175,5 +175,5 @@
         <parent link="base_link"/>
         <child link="femto_base"/>
-        <limit effort="1000.0" lower="0" upper="1.7" velocity="0.5"/>
+        <limit effort="1000.0" lower="0" upper="2.0" velocity="0.5"/>
         <origin xyz="0.05 0 0" rpy="0 -1.5707963 0"/>
     </joint>

File: wpr2_description/urdf/torso.xacro (robot description, xacro)
@@ -54,5 +54,5 @@
     <parent link="chest_link"/>
     <child link="femto_base"/>
-    <limit effort="1000.0" lower="0" upper="0.1" velocity="0.5"/>
+    <limit effort="1000.0" lower="0" upper="1.0" velocity="0.5"/>
     <origin xyz="0.05 0 0" rpy="0 -1.5707963 0"/>
   </joint>

File: wpr2_moveit_config/config/gazebo_wpr2.urdf (robot description, URDF)
Before this commit: robot wpr2, 32 links, 31 joints
Joints:
- joint femto_height: limit lower=0 upper=0.1 effort=1000.0 velocity=0.5 -> lower=0 upper=1.0 effort=1000.0 velocity=0.5
