Commit message: updata params

File: wpr2_description/urdf/torso.xacro (robot description, xacro)
@@ -54,5 +54,5 @@
     <parent link="chest_link"/>
     <child link="femto_base"/>
-    <limit effort="1000.0" lower="0" upper="1.0" velocity="0.5"/>
+    <limit effort="1000.0" lower="-1.0" upper="1.0" velocity="0.5"/>
     <origin xyz="0.05 0 0" rpy="0 -1.5707963 0"/>
   </joint>
