Commit message: update urdf

File: wpr2_description/urdf/arm_left.urdf.xacro (robot description, xacro)
@@ -67,5 +67,5 @@
       <parent link="left_link_1"/>
       <child link="left_link_2"/>
-      <origin xyz="0 0 0 " rpy="0 0 0"/>
+      <origin xyz="0 0 0 " rpy="0 ${M_PI} 0"/>
       <axis xyz="1 0 0"/>
     </joint>
@@ -86,5 +86,5 @@
           <mesh filename="package://wpr2_description/meshes/arm/arm_link_3.dae" scale="1 1 1"/>
         </geometry>
-        <origin xyz="0 0.19 0" rpy="${M_PI*0.5} 0 ${-M_PI*0.5}" />
+        <origin xyz="0 0.19 0" rpy="${-M_PI*0.5} 0 ${-M_PI*0.5}" />
       </visual>
       <collision>
@@ -137,5 +137,5 @@
       <parent link="left_link_3"/>
       <child link="left_link_4"/>
-      <origin xyz="0 0.19 0" rpy="0 ${M_PI} 0"/>
+      <origin xyz="0 0.19 0" rpy="0 0 0"/>
       <axis xyz="0 0 1"/>
     </joint>

File: wpr2_description/urdf/arm_right.urdf.xacro (robot description, xacro)
@@ -67,5 +67,5 @@
       <parent link="right_link_1"/>
       <child link="right_link_2"/>
-      <origin xyz="0 0 0 " rpy="0 0 0"/>
+      <origin xyz="0 0 0 " rpy="0 ${M_PI} 0"/>
       <axis xyz="1 0 0"/>
     </joint>
@@ -86,5 +86,5 @@
           <mesh filename="package://wpr2_description/meshes/arm/arm_link_3.dae" scale="1 1 1"/>
         </geometry>
-        <origin xyz="0 0.19 0" rpy="${-M_PI*0.5} 0 ${-M_PI*0.5}" />
+        <origin xyz="0 0.19 0" rpy="${M_PI*0.5} 0 ${-M_PI*0.5}" />
       </visual>
       <collision>
@@ -137,5 +137,5 @@
       <parent link="right_link_3"/>
       <child link="right_link_4"/>
-      <origin xyz="0 0.19 0" rpy="0 0 0"/>
+      <origin xyz="0 0.19 0" rpy="0 ${M_PI} 0"/>
       <axis xyz="0 0 1"/>
     </joint>

Commit message: add moveit

File: wpr2_description/urdf/arm_left.urdf.xacro (robot description, xacro)
@@ -51,5 +51,5 @@
           <mesh filename="package://wpr2_description/meshes/arm/arm_link_2.dae" scale="1 1 1"/>
         </geometry>
-        <origin rpy="${M_PI} 0 0" xyz="0 0 0"/>
+        <origin rpy="${M_PI} ${M_PI} 0" xyz="0 0 0"/>
       </visual>
       <collision>
@@ -91,5 +91,5 @@
         <origin xyz="0 0.19 0" rpy="0 0 0"/>
         <geometry>
-          <cylinder length="0.07" radius="0.041"/>
+          <cylinder length="0.12" radius="0.041"/>
         </geometry>
       </collision>
@@ -161,5 +161,5 @@
         <origin xyz="0 0 0" rpy="0 0 0"/>
         <geometry>
-          <cylinder length="0.07" radius="0.041"/>
+          <cylinder length="0.12" radius="0.041"/>
         </geometry>
       </collision>
@@ -266,4 +266,31 @@
       <mimic joint="left_finger_joint" multiplier="1" offset="0"/>
     </joint> -->
+    <!-- TCP(Tool Center Point) -->
+    <link name="left_tcp_link">
+      <inertial>
+        <mass value="0.001" />
+        <origin xyz="0 0 0" rpy="0 0 0" />
+        <inertia ixx="0.0001" ixy="0" ixz="0" iyy="0.0001" iyz="0" izz="0.0001" />
+      </inertial>
+      <!-- 手爪根部 -->
+      <collision>
+        <origin rpy = "0 0 0" xyz = "0.0 -0.13 0.0"/>
+        <geometry>
+            <box size="0.08 0.05 0.1"/>
+        </geometry>
+      </collision>
+       <!-- 手指活动范围 -->
+      <collision>
+        <origin rpy = "0 0 0" xyz = "0.0 -0.028 0.0"/>
+        <geometry>
+            <box size="0.18 0.15 0.04"/>
+        </geometry>
+      </collision>
+    </link>
+    <joint name="left_tcp_joint" type="fixed">
+      <parent link="left_link_6" />
+      <child link="left_tcp_link" />
+      <origin xyz="0 0.2 0" rpy="0 0 0" />
+    </joint>
   </xacro:macro>
 </robot>

File: wpr2_description/urdf/arm_right.urdf.xacro (robot description, xacro)
@@ -51,5 +51,5 @@
           <mesh filename="package://wpr2_description/meshes/arm/arm_link_2.dae" scale="1 1 1"/>
         </geometry>
-        <origin rpy="${M_PI} 0 0" xyz="0 0 0"/>
+        <origin rpy="${M_PI} ${M_PI} 0" xyz="0 0 0"/>
       </visual>
       <collision>
@@ -91,5 +91,5 @@
         <origin xyz="0 0.19 0" rpy="0 0 0"/>
         <geometry>
-          <cylinder length="0.07" radius="0.041"/>
+          <cylinder length="0.12" radius="0.041"/>
         </geometry>
       </collision>
@@ -161,5 +161,5 @@
         <origin xyz="0 0 0" rpy="0 0 0"/>
         <geometry>
-          <cylinder length="0.07" radius="0.041"/>
+          <cylinder length="0.12" radius="0.041"/>
         </geometry>
       </collision>
@@ -266,4 +266,31 @@
       <mimic joint="right_finger_joint" multiplier="1" offset="0"/>
     </joint> -->
+    <!-- TCP(Tool Center Point) -->
+    <link name="right_tcp_link">
+      <inertial>
+        <mass value="0.001" />
+        <origin xyz="0 0 0" rpy="0 0 0" />
+        <inertia ixx="0.0001" ixy="0" ixz="0" iyy="0.0001" iyz="0" izz="0.0001" />
+      </inertial>
+      <!-- 手爪根部 -->
+      <collision>
+        <origin rpy = "0 0 0" xyz = "0.0 -0.13 0.0"/>
+        <geometry>
+            <box size="0.08 0.05 0.1"/>
+        </geometry>
+      </collision>
+       <!-- 手指活动范围 -->
+      <collision>
+        <origin rpy = "0 0 0" xyz = "0.0 -0.028 0.0"/>
+        <geometry>
+            <box size="0.18 0.15 0.04"/>
+        </geometry>
+      </collision>
+    </link>
+    <joint name="right_tcp_joint" type="fixed">
+      <parent link="right_link_6" />
+      <child link="right_tcp_link" />
+      <origin xyz="0 0.2 0" rpy="0 0 0" />
+    </joint>
   </xacro:macro>
 </robot>

File: wpr2_description/urdf/base_mecanum.urdf.xacro (robot description, xacro)
@@ -4,4 +4,7 @@
   <xacro:property name="length" value="0.395"/>
   <xacro:property name="width" value="0.37"/>
+  <material name="black">
+    <color rgba="0 0 0 1"/>
+  </material>
   <!-- base_footprint -->
   <link name="base_footprint">
@@ -22,13 +25,42 @@
   <link name="base_link">
       <visual>
-          <geometry>
-              <mesh filename="package://wpr2_description/meshes/base.dae" scale="1 1 1"/>
-          </geometry>
+        <geometry>
+            <mesh filename="package://wpr2_description/meshes/base.dae" scale="1 1 1"/>
+        </geometry>
         <origin rpy = "0 0 0" xyz = "0.0 0.0 0.13"/>
       </visual>
-      <collision>
-        <origin xyz="0.005 0 0.05" rpy="0 0 0" />
-        <geometry>
-          <box size="0.57 0.37 0.1"/>
+      <visual>
+        <geometry>
+            <box size="0.02 0.32 0.2"/>
+        </geometry>
+        <origin rpy = "0 0 0" xyz = "-0.13 0.0 1.0"/>
+        <material name="black" />
+      </visual>
+      <!-- 底盘碰撞体 -->
+      <collision>
+        <origin xyz="0.005 0 0.07" rpy="0 0 0" />
+        <geometry>
+          <box size="0.57 0.46 0.12"/>
+        </geometry>
+      </collision>
+      <!-- 上舱盖 -->
+      <collision>
+        <origin xyz="-0.03 0 0.20" rpy="0 0 0" />
+        <geometry>
+          <box size="0.50 0.37 0.04"/>
+        </geometry>
+      </collision>
+      <!-- 立柱 -->
+      <collision>
+        <origin xyz="-0.07 0 0.68" rpy="0 0 0" />
+        <geometry>
+          <box size="0.10 0.20 0.90"/>
+        </geometry>
+      </collision>
+      <!-- 屏幕 -->
+      <collision>
+        <origin rpy = "0 0 0" xyz = "-0.13 0.0 1.0"/>
+        <geometry>
+            <box size="0.02 0.32 0.2"/>
         </geometry>
       </collision>

File: wpr2_description/urdf/torso.xacro (robot description, xacro)
@@ -9,7 +9,7 @@
     </visual>
     <collision>
-      <origin xyz="0.03 0 -0.01" rpy="0 0 0"/>
+      <origin xyz="0.04 0 -0.01" rpy="0 0 0"/>
       <geometry>
-       <box size="0.1 0.22 0.13"/>
+       <box size="0.1 0.22 0.15"/>
       </geometry>
     </collision>

Commit message: update for grippers

File: wpr2_description/urdf/arm_left.urdf.xacro (robot description, xacro)
@@ -1,4 +1,7 @@
 <?xml version="1.0"?>
 <robot xmlns:xacro="http://ros.org/wiki/xacro">
+  <material name="TransparentGreen">
+    <color rgba="0.0 1.0 0.0 0.5"/>
+  </material>
   <xacro:macro name="arm_left" params="base_frame x y z roll pitch yaw">
     <!-- joint 0 -->
@@ -185,9 +188,9 @@
       </actuator>
     </transmission>
-    <!-- joint 6 palm -->
+    <!-- joint 6 -->
     <link name="left_link_6">
       <visual>
         <geometry>
-          <mesh filename="package://wpr2_description/meshes/arm/arm_link_palm.dae" scale="1 1 1"/>
+          <mesh filename="package://wpr2_description/meshes/arm/arm_link_wrist.dae" scale="1 1 1"/>
         </geometry>
         <origin rpy="${-M_PI*0.5} ${M_PI*0.5}  0" xyz="0 0 0.05"/>
@@ -214,56 +217,83 @@
       </actuator>
     </transmission>
-    <link name="left_link_finger">
-      <visual>
-        <geometry>
-          <mesh filename="package://wpr2_description/meshes/arm/arm_link_palm.dae" scale="1 1 1"/>
-        </geometry>
-        <origin rpy="${-M_PI*0.5} ${-M_PI*0.5} 0" xyz="0 0 -0.05"/>
-      </visual>
-      <inertial>
-        <mass value="0.1"/>
-        <inertia ixx="0.1" ixy="0.0" ixz="0.0" iyy="0.1" iyz="0.0" izz="0.01"/>
-      </inertial>
-    </link>
-    <joint name="left_joint_finger" type="fixed">
+    <link name="left_link_knuckle_1">
+      <visual>
+        <geometry>
+          <mesh filename="package://wpr2_description/meshes/arm/arm_link_knuckle.dae" scale="1 1 1"/>
+        </geometry>
+        <origin rpy="${-M_PI*0.5} ${M_PI*0.5} 0" xyz="0 0 0"/>
+      </visual>
+      <inertial>
+        <mass value="0.1"/>
+        <inertia ixx="0.1" ixy="0.0" ixz="0.0" iyy="0.1" iyz="0.0" izz="0.01"/>
+      </inertial>
+    </link>
+    <joint name="left_joint_finger" type="revolute">
       <parent link="left_link_6"/>
-      <child link="left_link_finger"/>
-      <origin xyz="0 0 0" rpy="0 0 0"/>
-    </joint>
-    <!-- finger 0-->
-    <!-- <link name="left_finger_0">
-      <visual>
-        <geometry>
-          <box size="0.02 0.02 0.08"/>
-        </geometry>
-        <origin rpy="0 0 0" xyz="0 0 -0.04"/>
-        <material name="white"/>
-      </visual>
-    </link>
-    <joint name="left_finger_joint" type="prismatic">
-      <parent link="left_link_5"/>
-      <child link="left_finger_0"/>
-      <origin xyz="0 0 -0.325"/>
-      <axis xyz="0 1 0"/>
-      <limit effort="1000.0" lower="0" upper="0.05" velocity="0.5"/>
-    </joint> -->
-    <!-- finger 1-->
-    <!-- <link name="left_finger_1">
-      <visual>
-        <geometry>
-          <box size="0.02 0.02 0.08"/>
-        </geometry>
-        <origin rpy="0 0 0" xyz="0 0 -0.04"/>
-        <material name="white"/>
-      </visual>
-    </link>
-    <joint name="left_finger_joint_1" type="prismatic">
-      <parent link="left_link_5"/>
-      <child link="left_finger_1"/>
-      <origin xyz="0 0 -0.325"/>
-      <axis xyz="0 -1 0"/>
-      <limit effort="1000.0" lower="0" upper="0.05" velocity="0.5"/>
-      <mimic joint="left_finger_joint" multiplier="1" offset="0"/>
-    </joint> -->
+      <child link="left_link_knuckle_1"/>
+      <origin xyz="0.005 0.11 0" rpy="0 0 0"/>
+      <axis xyz="0 0 -1"/>
+      <limit effort="1000.0" lower="0" upper="1.57" velocity="0.5"/>
+    </joint>
+    <link name="left_link_tip_1">
+      <visual>
+        <geometry>
+          <mesh filename="package://wpr2_description/meshes/arm/arm_link_tip.dae" scale="1 1 1"/>
+        </geometry>
+        <origin rpy="${-M_PI*0.5} ${M_PI*0.5} 0" xyz="0 0 0"/>
+      </visual>
+      <inertial>
+        <mass value="0.1"/>
+        <inertia ixx="0.1" ixy="0.0" ixz="0.0" iyy="0.1" iyz="0.0" izz="0.01"/>
+      </inertial>
+    </link>
+    <joint name="left_joint_tip_1" type="revolute">
+      <parent link="left_link_knuckle_1"/>
+      <child link="left_link_tip_1"/>
+      <origin xyz="0 0.095 0" rpy="0 0 0"/>
+      <axis xyz="0 0 1"/>
+      <limit effort="1000.0" lower="0" upper="1.57" velocity="0.5"/>
+      <mimic joint="left_joint_finger" multiplier="1" offset="0"/>
+    </joint>
+    <link name="left_link_knuckle_2">
+      <visual>
+        <geometry>
+          <mesh filename="package://wpr2_description/meshes/arm/arm_link_knuckle.dae" scale="1 1 1"/>
+        </geometry>
+        <origin rpy="${-M_PI*0.5} ${-M_PI*0.5} 0" xyz="0 0 0"/>
+      </visual>
+      <inertial>
+        <mass value="0.1"/>
+        <inertia ixx="0.1" ixy="0.0" ixz="0.0" iyy="0.1" iyz="0.0" izz="0.01"/>
+      </inertial>
+    </link>
+    <joint name="left_joint_finger_2" type="revolute">
+      <parent link="left_link_6"/>
+      <child link="left_link_knuckle_2"/>
+      <origin xyz="-0.005 0.11 0" rpy="0 0 0"/>
+      <axis xyz="0 0 1"/>
+      <limit effort="1000.0" lower="0" upper="1.57" velocity="0.5"/>
+      <mimic joint="left_joint_finger" multiplier="1" offset="0"/>
+    </joint>
+    <link name="left_link_tip_2">
+      <visual>
+        <geometry>
+          <mesh filename="package://wpr2_description/meshes/arm/arm_link_tip.dae" scale="1 1 1"/>
+        </geometry>
+        <origin rpy="${-M_PI*0.5} ${M_PI*0.5} 0" xyz="0 0 0"/>
+      </visual>
+      <inertial>
+        <mass value="0.1"/>
+        <inertia ixx="0.1" ixy="0.0" ixz="0.0" iyy="0.1" iyz="0.0" izz="0.01"/>
+      </inertial>
+    </link>
+    <joint name="left_joint_tip_2" type="revolute">
+      <parent link="left_link_knuckle_2"/>
+      <child link="left_link_tip_2"/>
+      <origin xyz="0 0.095 0" rpy="0 0 0"/>
+      <axis xyz="0 0 -1"/>
+      <limit effort="1000.0" lower="0" upper="1.57" velocity="0.5"/>
+      <mimic joint="left_joint_finger" multiplier="1" offset="0"/>
+    </joint>
     <!-- TCP(Tool Center Point) -->
     <link name="left_tcp_link">

File: wpr2_description/urdf/arm_right.urdf.xacro (robot description, xacro)
@@ -185,9 +185,9 @@
       </actuator>
     </transmission>
-    <!-- joint 6 palm -->
+    <!-- joint 6 -->
     <link name="right_link_6">
       <visual>
         <geometry>
-          <mesh filename="package://wpr2_description/meshes/arm/arm_link_palm.dae" scale="1 1 1"/>
+          <mesh filename="package://wpr2_description/meshes/arm/arm_link_wrist.dae" scale="1 1 1"/>
         </geometry>
         <origin rpy="${-M_PI*0.5} ${M_PI*0.5}  0" xyz="0 0 0.05"/>
@@ -214,56 +214,83 @@
       </actuator>
     </transmission>
-    <link name="right_link_finger">
-      <visual>
-        <geometry>
-          <mesh filename="package://wpr2_description/meshes/arm/arm_link_palm.dae" scale="1 1 1"/>
-        </geometry>
-        <origin rpy="${-M_PI*0.5} ${-M_PI*0.5} 0" xyz="0 0 -0.05"/>
-      </visual>
-      <inertial>
-        <mass value="0.1"/>
-        <inertia ixx="0.1" ixy="0.0" ixz="0.0" iyy="0.1" iyz="0.0" izz="0.01"/>
-      </inertial>
-    </link>
-    <joint name="right_joint_finger" type="fixed">
+    <link name="right_link_knuckle_1">
+      <visual>
+        <geometry>
+          <mesh filename="package://wpr2_description/meshes/arm/arm_link_knuckle.dae" scale="1 1 1"/>
+        </geometry>
+        <origin rpy="${-M_PI*0.5} ${M_PI*0.5} 0" xyz="0 0 0"/>
+      </visual>
+      <inertial>
+        <mass value="0.1"/>
+        <inertia ixx="0.1" ixy="0.0" ixz="0.0" iyy="0.1" iyz="0.0" izz="0.01"/>
+      </inertial>
+    </link>
+    <joint name="right_joint_finger" type="revolute">
       <parent link="right_link_6"/>
-      <child link="right_link_finger"/>
-      <origin xyz="0 0 0" rpy="0 0 0"/>
-    </joint>
-    <!-- finger 0-->
-    <!-- <link name="right_finger_0">
-      <visual>
-        <geometry>
-          <box size="0.02 0.02 0.08"/>
-        </geometry>
-        <origin rpy="0 0 0" xyz="0 0 -0.04"/>
-        <material name="white"/>
-      </visual>
-    </link>
-    <joint name="right_finger_joint" type="prismatic">
-      <parent link="right_link_5"/>
-      <child link="right_finger_0"/>
-      <origin xyz="0 0 -0.325"/>
-      <axis xyz="0 1 0"/>
-      <limit effort="1000.0" lower="0" upper="0.05" velocity="0.5"/>
-    </joint> -->
-    <!-- finger 1-->
-    <!-- <link name="right_finger_1">
-      <visual>
-        <geometry>
-          <box size="0.02 0.02 0.08"/>
-        </geometry>
-        <origin rpy="0 0 0" xyz="0 0 -0.04"/>
-        <material name="white"/>
-      </visual>
-    </link>
-    <joint name="right_finger_joint_1" type="prismatic">
-      <parent link="right_link_5"/>
-      <child link="right_finger_1"/>
-      <origin xyz="0 0 -0.325"/>
-      <axis xyz="0 -1 0"/>
-      <limit effort="1000.0" lower="0" upper="0.05" velocity="0.5"/>
-      <mimic joint="right_finger_joint" multiplier="1" offset="0"/>
-    </joint> -->
+      <child link="right_link_knuckle_1"/>
+      <origin xyz="0.005 0.11 0" rpy="0 0 0"/>
+      <axis xyz="0 0 -1"/>
+      <limit effort="1000.0" lower="0" upper="1.57" velocity="0.5"/>
+    </joint>
+    <link name="right_link_tip_1">
+      <visual>
+        <geometry>
+          <mesh filename="package://wpr2_description/meshes/arm/arm_link_tip.dae" scale="1 1 1"/>
+        </geometry>
+        <origin rpy="${-M_PI*0.5} ${M_PI*0.5} 0" xyz="0 0 0"/>
+      </visual>
+      <inertial>
+        <mass value="0.1"/>
+        <inertia ixx="0.1" ixy="0.0" ixz="0.0" iyy="0.1" iyz="0.0" izz="0.01"/>
+      </inertial>
+    </link>
+    <joint name="right_joint_tip_1" type="revolute">
+      <parent link="right_link_knuckle_1"/>
+      <child link="right_link_tip_1"/>
+      <origin xyz="0 0.095 0" rpy="0 0 0"/>
+      <axis xyz="0 0 1"/>
+      <limit effort="1000.0" lower="0" upper="1.57" velocity="0.5"/>
+      <mimic joint="right_joint_finger" multiplier="1" offset="0"/>
+    </joint>
+    <link name="right_link_knuckle_2">
+      <visual>
+        <geometry>
+          <mesh filename="package://wpr2_description/meshes/arm/arm_link_knuckle.dae" scale="1 1 1"/>
+        </geometry>
+        <origin rpy="${-M_PI*0.5} ${-M_PI*0.5} 0" xyz="0 0 0"/>
+      </visual>
+      <inertial>
+        <mass value="0.1"/>
+        <inertia ixx="0.1" ixy="0.0" ixz="0.0" iyy="0.1" iyz="0.0" izz="0.01"/>
+      </inertial>
+    </link>
+    <joint name="right_joint_finger_2" type="revolute">
+      <parent link="right_link_6"/>
+      <child link="right_link_knuckle_2"/>
+      <origin xyz="-0.005 0.11 0" rpy="0 0 0"/>
+      <axis xyz="0 0 1"/>
+      <limit effort="1000.0" lower="0" upper="1.57" velocity="0.5"/>
+      <mimic joint="right_joint_finger" multiplier="1" offset="0"/>
+    </joint>
+    <link name="right_link_tip_2">
+      <visual>
+        <geometry>
+          <mesh filename="package://wpr2_description/meshes/arm/arm_link_tip.dae" scale="1 1 1"/>
+        </geometry>
+        <origin rpy="${-M_PI*0.5} ${M_PI*0.5} 0" xyz="0 0 0"/>
+      </visual>
+      <inertial>
+        <mass value="0.1"/>
+        <inertia ixx="0.1" ixy="0.0" ixz="0.0" iyy="0.1" iyz="0.0" izz="0.01"/>
+      </inertial>
+    </link>
+    <joint name="right_joint_tip_2" type="revolute">
+      <parent link="right_link_knuckle_2"/>
+      <child link="right_link_tip_2"/>
+      <origin xyz="0 0.095 0" rpy="0 0 0"/>
+      <axis xyz="0 0 -1"/>
+      <limit effort="1000.0" lower="0" upper="1.57" velocity="0.5"/>
+      <mimic joint="right_joint_finger" multiplier="1" offset="0"/>
+    </joint>
     <!-- TCP(Tool Center Point) -->
     <link name="right_tcp_link">
